File: Hardware/KiCAD_Project_Files/LaunchPad_3x7-Segment_Display_Booster_Pack.sch (KiCad schematic (older format))
At the start: 17 parts, among them P1 CONN_10, P2 CONN_10, U1 74LS125, U2 LTC4624JF

Commit message: Updated to current board design
Parts:
- removed P1, P2: CONN_10, symbol CONN_10
- removed R1, R2, R3, R4: 1k, symbol R
- removed R10, R11, R12, R5, R6, R7, R8, R9: 100, symbol R
- removed U2: LTC4624JF, symbol LTC4624JF
- added P1, P2: HEADER_1X10, symbol HEADER_1X10
- added R1, R10, R11, R12, R2, R3, R4, R5, R6, R7, R8, R9: RES, symbol RES
- added unit 5 of U1
- added U2: LTC4624, symbol LTC4624
Connections:
- net labels added: +3.3V
- net labels removed: VCC
- wire segments 94 -> 95
Other:
- note added: "2"
- note removed: "B"
- moved on the sheet: C1, U1A, U1B, U1C, U1D
