File: Hardware/KiCAD_Project_Files/LaunchPad_3x7-Segment_Display_Booster_Pack.sch (KiCad schematic (older format))
At the start: 17 parts, among them P1 HEADER_1X10, P2 HEADER_1X10, U1 74LS125, U2 LTC4624

Commit message: Updated to new kicad board format. + Rendered pic + pdf of BOM
Minor corrections to schematic.
Connections:
- net labels added: DISP_SEG_A, DISP_SEG_B, DISP_SEG_C, DISP_SEG_D, DISP_SEG_DP, DISP_SEG_E, DISP_SEG_F, DISP_SEG_G
- wire segments 95 -> 87
Other:
- moved on the sheet: C1, R10, R11, R12, R5, R6, R7, R8, R9, U1E

Commit message: Minor changes to schematic due to updtaed female header decal. Updated sheet size to standard 8.5x11. Moved BOM's and Schematic into respective folders to conform to newer project directory structure.
Other:
- note removed: "1"
- note removed: "LaunchPad 3x7-Segment Display Booster Pack"
- moved on the sheet: C1, R1, R10, R11, R12, R2, R3, R4, R5, R6, R7, R8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
